Commit message: quadruped working

File: body.urdf (robot description, URDF)
Before this commit: robot robot, 9 links, 8 joints
Links:
- link BackLeg: geometry collision box size=0.2 0.5 0.2; visual box size=0.2 0.5 0.2
- link BackLowerLeg: geometry collision box size=0.2 0.2 0.75; visual box size=0.2 0.2 0.75
- link FrontLeg: geometry collision box size=0.2 0.5 0.2; visual box size=0.2 0.5 0.2
- link FrontLowerLeg: geometry collision box size=0.2 0.2 0.75; visual box size=0.2 0.2 0.75
- link LeftLeg: geometry collision box size=0.5 0.2 0.2; visual box size=0.5 0.2 0.2
- link LeftLowerLeg: geometry collision box size=0.2 0.2 0.75; visual box size=0.2 0.2 0.75
- link RightLeg: geometry collision box size=0.5 0.2 0.2; visual box size=0.5 0.2 0.2
- link RightLowerLeg: geometry collision box size=0.2 0.2 0.75; visual box size=0.2 0.2 0.75
Joints:
- joint BackLeg_BackLowerLeg: origin xyz=0 -1 0 rpy=0 0 0 -> xyz=0 -0.5 0 rpy=0 0 0
- joint FrontLeg_FrontLowerLeg: origin xyz=0 1 0 rpy=0 0 0 -> xyz=0 0.5 0 rpy=0 0 0
- joint LeftLeg_LeftLowerLeg: origin xyz=-1 0 0 rpy=0 0 0 -> xyz=-0.5 0 0 rpy=0 0 0
- joint RightLeg_RightLowerLeg: origin xyz=1 0 0 rpy=0 0 0 -> xyz=0.5 0 0 rpy=0 0 0

Commit message: quadruped working

File: body.urdf (robot description, URDF)
Before this commit: robot robot, 9 links, 8 joints
Links:
- link BackLeg: geometry collision box size=0.2 0.3 0.2; visual box size=0.2 0.3 0.2
- link FrontLeg: geometry collision box size=0.2 0.3 0.2; visual box size=0.2 0.3 0.2
- link LeftLeg: geometry collision box size=0.3 0.2 0.2; visual box size=0.3 0.2 0.2
- link RightLeg: geometry collision box size=0.3 0.2 0.2; visual box size=0.3 0.2 0.2
Joints:
- joint BackLeg_BackLowerLeg: origin xyz=0 -0.5 0 rpy=0 0 0 -> xyz=0 -0.3 0 rpy=0 0 0
- joint FrontLeg_FrontLowerLeg: origin xyz=0 0.5 0 rpy=0 0 0 -> xyz=0 0.3 0 rpy=0 0 0
- joint LeftLeg_LeftLowerLeg: origin xyz=-0.5 0 0 rpy=0 0 0 -> xyz=-0.3 0 0 rpy=0 0 0
- joint RightLeg_RightLowerLeg: origin xyz=0.5 0 0 rpy=0 0 0 -> xyz=0.3 0 0 rpy=0 0 0
